File: BRM.kicad_sch (KiCad schematic)
At the start: 31 parts, among them J1 2606-1102, J2 2601-1108, J4 2601-1108

Commit message: VRM work
Changed lines of the file:
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@@
 			)
 		)
-		(pin "GND" input
+		(pin "GND" passive
 			(at 148.59 57.15 90)
 			(effects
@@
 			)
 		)
-		(pin "Vout" input
+		(pin "Vout" output
 			(at 160.02 63.5 0)
 			(effects
