File: VRM.kicad_sch (KiCad schematic)
At the start: 17 parts, among them U1 TPS55289RYQR

Commit message: VRM work
Changed lines of the file:
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@@
 		(pin "6"
+		)
+		(pin "21"
 		)
 		(instances
